File: led-strip-esphome/_autosave-led-strip-esphome.kicad_pcb (KiCad board)
At the start: 2 copper layers, 2 parts, among them U1 TP4056_C725790

Commit message: pcb
Parts:
- added D2: LED, LED_SMD:LED_0603_1608Metric, F.Cu at (133.9, 85.5)
- added D3: LED, LED_SMD:LED_0603_1608Metric, F.Cu at (133.9, 88.1)
- added USB1: TYPE-C 6P(073), easyeda2kicad:TYPE-C-SMD_TYPE-C-6P_5, F.Cu at (140.5, 77.4)
Connections:
- U1 pad 1: unconnected-(U1-TEMP-Pad1) -> GND
- U1 pad 2: unconnected-(U1-PROG-Pad2) -> Net-(U1-PROG)
- U1 pad 3: unconnected-(U1-GND-Pad3) -> GND
- U1 pad 4: unconnected-(U1-VCC-Pad4) -> Net-(D2-A)
- U1 pad 5: unconnected-(U1-BAT-Pad5) -> Net-(BT1-+)
- U1 pad 6: unconnected-(U1-~{STDBY}-Pad6) -> Net-(U1-~{STDBY})
- U1 pad 7: unconnected-(U1-~{CHRG}-Pad7) -> Net-(U1-~{CHRG})
- U1 pad 8: unconnected-(U1-CE-Pad8) -> Net-(D2-A)
