File: led-strip-esphome/_autosave-led-strip-esphome.kicad_sch (KiCad schematic)
At the start: 16 parts, among them U1 TP4056_C725790

Commit message: pcb
Parts:
- added C3: RVT1E221M0607_C2918361, easyeda2kicad:CAP-SMD_BD6.3-L6.6-W6.6-LS7.4-FD, symbol easyeda2kicad:RVT1E221M0607_C2918361
- added C4, C5, C6, C7, C8: 22uF, symbol Device:C
- added D5: 1N5824_C7503125, easyeda2kicad:DO-27_BD5.3-L8.4-P12.40-D1.3-RD, symbol easyeda2kicad:1N5824_C7503125
- added L1: 33uh, symbol Device:L
- added L2: 3.3uh, symbol Device:L
- added R8: 33k, symbol Device:R
- added R9: 100k, symbol Device:R
- added U2: LM2596S-3.3, Package_TO_SOT_SMD:TO-263-5_TabPin3, symbol Regulator_Switching:LM2596S-3.3
- added U3: RVT1E681M1010_C5221838, easyeda2kicad:CAP-SMD_BD10.0-L10.3-W10.3-LS11.6-FD, symbol easyeda2kicad:RVT1E681M1010_C5221838
- added U4: AP2007SPER, easyeda2kicad:ESOP-8_L4.9-W3.9-P1.27-LS6.0-BL-EP, symbol easyeda2kicad:AP2007SPER
- D1: LCSC (none) -> C7423443
Connections:
- net 3V~4.2V Out: now also C4.1, C5.1, L2.1, U4.3 (VIN), U4.4 (EN)
- net GND: now also C2.1, D2.2 (A), D3.2 (A), R4.2, U1.4 (VCC), U1.8 (CE), C3.2, C4.2, C5.2, C6.2, C7.2, C8.2, D5.2 (A), R8.2, U2.3 (GND), U2.5 (~{ON}/OFF), U3.2, U4.5 (GND)
- new net: C6.1, C7.1, C8.1, R9.1, U2.1 (VIN), U3.1, U4.7 (VOUT), U4.8 (VOUT)
- new net: R8.1, R9.2
- new net: D5.1 (K), L1.1, U2.2 (OUT)
- new net: C3.1, L1.2, U2.4 (FB)
- new net: L2.2, U4.1 (LX), U4.2 (LX)
Other:
- moved on the sheet: BT1, C1, C2, D1, D2, D3, D4, R1, R2, R3, R4, R5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
