File: led-strip-esphome/led-strip-esphome.kicad_sch (KiCad schematic)
At the start: 4 parts, among them U1 TP4056_C725790

Commit message: pcb
Parts:
- removed TH1: Thermistor_NTC, symbol Device:Thermistor_NTC
- added C1, C2: 10uF, symbol Device:C
- added C3: RVT1E221M0607_C2918361, easyeda2kicad:CAP-SMD_BD6.3-L6.6-W6.6-LS7.4-FD, symbol easyeda2kicad:RVT1E221M0607_C2918361
- added C4, C5, C6, C7, C8: 22uF, symbol Device:C
- added D2, D3: LED, LED_SMD:LED_0603_1608Metric, symbol Device:LED
- added D4: D, symbol Device:D
- added D5: 1N5824_C7503125, easyeda2kicad:DO-27_BD5.3-L8.4-P12.40-D1.3-RD, symbol easyeda2kicad:1N5824_C7503125
- added L1: 33uh, symbol Device:L
- added L2: 3.3uh, symbol Device:L
- added R1: 2.4k, symbol Device:R
- added R2, R3: 210, symbol Device:R
- added R4: 0.4, symbol Device:R
- added R5: 1M, LED_SMD:LED_0805_2012Metric, symbol Device:R
- added R6, R7: 5.11k, symbol Device:R
- added R8: 33k, symbol Device:R
- added R9: 100k, symbol Device:R
- added U2: LM2596S-3.3, Package_TO_SOT_SMD:TO-263-5_TabPin3, symbol Regulator_Switching:LM2596S-3.3
- added U3: RVT1E681M1010_C5221838, easyeda2kicad:CAP-SMD_BD10.0-L10.3-W10.3-LS11.6-FD, symbol easyeda2kicad:RVT1E681M1010_C5221838
- added U4: AP2007SPER, easyeda2kicad:ESOP-8_L4.9-W3.9-P1.27-LS6.0-BL-EP, symbol easyeda2kicad:AP2007SPER
- added USB1: TYPE-C 6P(073), easyeda2kicad:TYPE-C-SMD_TYPE-C-6P_5, symbol easyeda2kicad:TYPE-C6P(073)
- D1: LCSC (none) -> C7423443
Connections:
- net at BT1.1 (+), U1.5 (BAT): now also C1.1
- net GND: now reaches BT1.2 (-)
- net GND: now also U1.1 (TEMP), U1.3 (GND), U1.4 (VCC), U1.8 (CE), C1.2, C2.1, C2.2, C3.2, C4.2, C5.2, C6.2, C7.2, C8.2, D2.2 (A), D3.2 (A), D5.2 (A), R1.2, R4.2, R5.2, R6.2, R7.2, R8.2, U2.3 (GND), U2.5 (~{ON}/OFF), U3.2, U4.5 (GND), USB1.A12 (GND), USB1.B12 (GND)
- net at U1.2 (PROG): now also R1.1
- net at U1.6 (~{STDBY}): now also R3.2
- net at U1.7 (~{CHRG}): now also R2.2
- new net: R5.1, USB1.7 (EH)
- new net: R6.1, USB1.A5 (CC1)
- new net: D4.2 (A), USB1.A9 (VBUS), USB1.B9 (VBUS)
- new net: R7.1, USB1.B5 (CC2)
- new net: C6.1, C7.1, C8.1, R9.1, U2.1 (VIN), U3.1, U4.7 (VOUT), U4.8 (VOUT)
- new net: R8.1, R9.2
- new net: D5.1 (K), L1.1, U2.2 (OUT)
- new net: C3.1, L1.2, U2.4 (FB)
- new net: D3.1 (K), R2.1
- new net: C4.1, C5.1
- new net: L2.2, U4.1 (LX), U4.2 (LX)
- new net: L2.1, U4.3 (VIN), U4.4 (EN)
- new net: D2.1 (K), R3.1
- new net 3V~4.2V Out: D4.1 (K), R4.1
- no-connect marks 0 -> 1
Other:
- moved on the sheet: BT1, D1, U1

Commit message: pcb
Parts:
- added C9: 0.1uF, Capacitor_SMD:CP_Elec_4x5.4, symbol Device:C_Polarized
- added Q1: FS8205A_C2830320, easyeda2kicad:SOT-23-6_L2.9-W1.6-P0.95-LS2.8-BR, symbol easyeda2kicad:FS8205A_C2830320
- added R10: 100, symbol Device:R
- added R11: 1k, symbol Device:R
- added U5: DW01A, Package_TO_SOT_SMD:SOT-23-6, symbol Battery_Management:DW01A
- added U6: AMS1117-3.3, Package_TO_SOT_SMD:SOT-223-3_TabPin2, symbol Regulator_Linear:AMS1117-3.3
Connections:
- net 3V~4.2V Out: now also U6.3 (VI)
- net GND: now also Q1.3 (S2), R11.2, U6.1 (GND); no longer BT1.2 (-), C1.2
- net at BT1.1 (+), C1.1, U1.5 (BAT): now also R10.2
- new net: BT1.2 (-), C1.2, C9.2, Q1.1 (S1), U5.6 (GND)
- new net: C9.1, R10.1, U5.5 (VCC)
- new net: Q1.4 (G2), U5.3 (OC)
- new net: Q1.6 (G1), U5.1 (OD)
- new net: R11.1, U5.2 (CS)
- no-connect marks 1 -> 3

Commit message: pcb
Parts:
- removed C3: RVT1E221M0607_C2918361, easyeda2kicad:CAP-SMD_BD6.3-L6.6-W6.6-LS7.4-FD, symbol easyeda2kicad:RVT1E221M0607_C2918361
- removed C5, C6, C7, C8: 22uF, symbol Device:C
- removed D5: 1N5824_C7503125, easyeda2kicad:DO-27_BD5.3-L8.4-P12.40-D1.3-RD, symbol easyeda2kicad:1N5824_C7503125
- removed L1: 33uh, symbol Device:L
- removed L2: 3.3uh, symbol Device:L
- removed R8: 33k, symbol Device:R
- removed R9: 100k, symbol Device:R
- removed U2: LM2596S-3.3, Package_TO_SOT_SMD:TO-263-5_TabPin3, symbol Regulator_Switching:LM2596S-3.3
- removed U3: RVT1E681M1010_C5221838, easyeda2kicad:CAP-SMD_BD10.0-L10.3-W10.3-LS11.6-FD, symbol easyeda2kicad:RVT1E681M1010_C5221838
- removed U4: AP2007SPER, easyeda2kicad:ESOP-8_L4.9-W3.9-P1.27-LS6.0-BL-EP, symbol easyeda2kicad:AP2007SPER
- removed U6: AMS1117-3.3, Package_TO_SOT_SMD:SOT-223-3_TabPin2, symbol Regulator_Linear:AMS1117-3.3
- added C3: 1uF, symbol Device:C
- added U2: BL8072COTR33, easyeda2kicad:TO-252-3_L6.6-W6.1-P2.28-LS10.1-BL, symbol easyeda2kicad:BL8072COTR33
- added U3: AI-WB2-12F, easyeda2kicad:COMM-SMD_22P-L24.0-W16.0-P2.00_ZIGBEE, symbol easyeda2kicad:AI-WB2-12F
- C4: value 22uF -> 1uF
Connections:
- net 3V~4.2V Out: now also C3.1, U2.3 (VDD)
- net GND: now also C3.2, U2.1 (VSS)
- net at C4.1: now also U2.2 (OUT), U2.4 (OUT)

Commit message: pcb
Parts:
- added H1: PZ254V-11-04P_C2691448, easyeda2kicad:HDR-TH_4P-P2.54-V-M, symbol easyeda2kicad:PZ254V-11-04P_C2691448
Connections:
- net GND: now also U3.9 (GND), H1.4
- net at U3.15 (RXD): now also H1.3
- net at U3.16 (TXD): now also H1.2
- net +3.3V: now reaches U3.8 (VCC)
- net +3.3V: now also C4.1, U2.2 (OUT), U2.4 (OUT), H1.1
Other:
- moved on the sheet: U3

Commit message: pcb
Parts:
- added D10, D11, D13, D14, D15, D16, D17, D18, D19, D5, D6, D7, D8, D9: LED, LED_SMD:LED_PLCC_2835, symbol Device:LED
Connections:
- net at D1.1 (K): now also D10.1 (K), D11.1 (K), D13.1 (K), D14.1 (K), D15.1 (K), D16.1 (K), D17.1 (K), D18.1 (K), D19.1 (K), D5.1 (K), D6.1 (K), D7.1 (K), D8.1 (K), D9.1 (K)
- net at D1.2 (A): now also D10.2 (A), D11.2 (A), D13.2 (A), D14.2 (A), D15.2 (A), D16.2 (A), D17.2 (A), D18.2 (A), D19.2 (A), D5.2 (A), D6.2 (A), D7.2 (A), D8.2 (A), D9.2 (A)
Other:
- moved on the sheet: D1

Commit message: schematic finished
Parts:
- added C5: 4.7uF, symbol Device:C
- added C6: 10uF, symbol Device:C
- added D12: D_Schottky, symbol Device:D_Schottky
- added L1: 10uH, symbol Device:L
- added R8: 0.25, symbol Device:R
- added U4: LGS63042, easyeda2kicad:SOT-23-5_L2.9-W1.6-P0.95-LS2.8-BL, symbol easyeda2kicad:LGS63042
Connections:
- net +3.3V: now also C5.2, C6.2, D12.1 (K), R8.2, U4.5 (VIN)
- net GND: now also C5.1, U4.2 (GND)
- net RX: now reaches H1.3, U3.15 (RXD)
- net TX: now reaches H1.2, U3.16 (TXD)
- net at U3.5 (IO14): now also U4.3 (EN)
- net at D1.1 (K), D10.1 (K), D11.1 (K)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: now also C6.1, L1.1
- net at D1.2 (A), D10.2 (A), D11.2 (A)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: now also R8.1, U4.4 (CSN)
- new net: D12.2 (A), L1.2, U4.1 (SW)
Other:
- moved on the sheet: H1

Commit message: add footprints
Parts:
- C1, C2, C6: footprint (none) -> Capacitor_SMD:C_0805_2012Metric
- D12: footprint (none) -> Diode_SMD:D_SMA; LCSC (none) -> C5350986
- L1: footprint (none) -> Inductor_SMD:L_Ferrocore_DLG-0403; LCSC (none) -> C2929419
Connections:
- net GND: now also C1.1; no longer C2.1, C2.2, D2.2 (A), D3.2 (A), R4.2, U1.4 (VCC), U1.8 (CE), USB1.A12 (GND), USB1.B12 (GND)
- net at BT1.1 (+), R10.2, U1.5 (BAT): now also C2.2; no longer C1.1
- net at BT1.2 (-), C9.2, Q1.1 (S1)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: now also C2.1; no longer C1.2
- new net: C1.2, D2.2 (A), D3.2 (A), R4.2, U1.4 (VCC), U1.8 (CE), USB1.A12 (GND), USB1.B12 (GND)

Commit message: add footprints
Parts:
- removed BT1: Battery_Cell, symbol Device:Battery_Cell
- added U6: XDM254-1-02-W-8.5-G0, easyeda2kicad:HDR-TH_2P-P2.54-H-F-W10.0-N, symbol easyeda2kicad:XDM254-1-02-W-8.5-G0
- D4: footprint (none) -> Diode_SMD:D_SMA; LCSC (none) -> C5154212
Connections:
- net +: now reaches C2.2, R10.2, U1.5 (BAT)
- net +: now also U6.1
- net at C2.1, C9.2, Q1.1 (S1)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: now also U6.2
Other:
- moved on the sheet: D4
Changed lines of the file:
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@@
 	(paper "A3")
 	(junction
-		(at 224.79 115.57)
+		(at 193.04 39.37)
 		(diameter 0)
 		(color 0 0 0 0)
 	)
 	(junction
-		(at 64.77 38.1)
+		(at 224.79 115.57)
 		(diameter 0)
 		(color 0 0 0 0)
 	)
 	(junction
-		(at 138.43 17.78)
+		(at 64.77 38.1)
 		(diameter 0)
 		(color 0 0 0 0)
@@
 	)
 	(junction
+		(at 138.43 16.51)
+		(diameter 0)
+		(color 0 0 0 0)
+	)
+	(junction
 		(at 179.07 46.99)
 		(diameter 0)
@@
 	)
 	(junction
-		(at 193.04 39.37)
-		(diameter 0)
-		(color 0 0 0 0)
-	)
-	(junction
 		(at 180.34 115.57)
 		(diameter 0)
@@
 	)
 	(junction
+		(at 193.04 46.99)
+		(diameter 0)
+		(color 0 0 0 0)
+	)
+	(junction
 		(at 199.39 107.95)
 		(diameter 0)
@@
 	)
 	(junction
-		(at 193.04 46.99)
-		(diameter 0)
-		(color 0 0 0 0)
-	)
-	(junction
 		(at 312.42 109.22)
 		(diameter 0)
@@
 	(wire
 		(pts
-			(xy 138.43 13.97) (xy 138.43 17.78)
-		)
-		(stroke
-			(width 0)
-			(type default)
-		)
-	)
-	(wire
-		(pts
 			(xy 256.54 68.58) (xy 228.6 68.58)
 		)
@@
 	(wire
 		(pts
-			(xy 121.92 17.78) (xy 121.92 27.94)
+			(xy 121.92 16.51) (xy 121.92 27.94)
 		)
 		(stroke
@@
 	(wire
 		(pts
-			(xy 138.43 19.05) (xy 138.43 17.78)
-		)
-		(stroke
-			(width 0)
-			(type default)
-		)
-	)
-	(wire
-		(pts
 			(xy 166.37 41.91) (xy 168.91 41.91)
 		)
@@
 	(wire
 		(pts
-			(xy 210.82 46.99) (xy 193.04 46.99)
+			(xy 55.88 33.02) (xy 57.15 33.02)
 		)
 		(stroke
@@
 	(wire
 		(pts
-			(xy 55.88 33.02) (xy 57.15 33.02)
+			(xy 270.51 16.51) (xy 270.51 20.32)
 		)
 		(stroke
@@
 	(wire
 		(pts
-			(xy 270.51 16.51) (xy 270.51 20.32)
+			(xy 218.44 31.75) (xy 218.44 46.99)
 		)
 		(stroke
@@
 	(wire
 		(pts
-			(xy 218.44 31.75) (xy 218.44 46.99)
+			(xy 312.42 109.22) (xy 314.96 109.22)
 		)
 		(stroke
@@
 	(wire
 		(pts
-			(xy 312.42 109.22) (xy 314.96 109.22)
+			(xy 148.59 134.62) (xy 148.59 107.95)
 		)
 		(stroke
@@
 	(wire
 		(pts
-			(xy 148.59 134.62) (xy 148.59 107.95)
+			(xy 172.72 30.48) (xy 173.99 30.48)
 		)
 		(stroke
@@
 	(wire
 		(pts
-			(xy 172.72 30.48) (xy 173.99 30.48)
+			(xy 193.04 44.45) (xy 193.04 46.99)
 		)
 		(stroke
@@
 	(wire
 		(pts
+			(xy 193.04 46.99) (xy 210.82 46.99)
+		)
+		(stroke
+			(width 0)
+			(type default)
+		)
+	)
+	(wire
+		(pts
 			(xy 332.74 101.6) (xy 332.74 113.03)
 		)
@@
 	(wire
 		(pts
-			(xy 130.81 57.15) (xy 130.81 41.91)
+			(xy 138.43 13.97) (xy 138.43 16.51)
 		)
 		(stroke
@@
 	(wire
 		(pts
-			(xy 238.76 107.95) (xy 245.11 107.95)
+			(xy 130.81 57.15) (xy 130.81 41.91)
 		)
 		(stroke
@@
 	(wire
 		(pts
-			(xy 251.46 134.62) (xy 251.46 128.27)
+			(xy 238.76 107.95) (xy 245.11 107.95)
 		)
 		(stroke
@@
 	(wire
 		(pts
-			(xy 304.8 114.3) (xy 308.61 114.3)
+			(xy 251.46 134.62) (xy 251.46 128.27)
 		)
 		(stroke
@@
 	(wire
 		(pts
-			(xy 121.92 17.78) (xy 120.65 17.78)
+			(xy 304.8 114.3) (xy 308.61 114.3)
 		)
 		(stroke
@@
 	(wire
 		(pts
-			(xy 128.27 17.78) (xy 138.43 17.78)
+			(xy 129.54 16.51) (xy 138.43 16.51)
 		)
 		(stroke
@@
 	(wire
 		(pts
+			(xy 138.43 16.51) (xy 138.43 19.05)
+		)
+		(stroke
+			(width 0)
+			(type default)
+		)
+	)
+	(wire
+		(pts
 			(xy 144.78 16.51) (xy 144.78 26.67)
 		)
@@
 	(wire
 		(pts
+			(xy 193.04 39.37) (xy 193.04 41.91)
+		)
+		(stroke
+			(width 0)
+			(type default)
+		)
+	)
+	(wire
+		(pts
 			(xy 330.2 88.9) (xy 330.2 116.84)
 		)
@@
 		)
 	)
+	(global_label "+"
+		(shape input)
+		(at 193.04 41.91 180)
+		(fields_autoplaced yes)
+		(effects
+			(font
+				(size 1.27 1.27)
+			)
+			(justify right)
+		)
+		(property "Intersheetrefs" "${INTERSHEET_REFS}"
+			(at 188.4824 41.91 0)
+			(effects
+				(font
+					(size 1.27 1.27)
+				)
+				(justify right)
+				(hide yes)
+			)
+		)
+	)
 	(global_label "VCC"
 		(shape input)
@@
 	)
 	(symbol
-		(lib_id "Device:Battery_Cell")
-		(at 193.04 44.45 0)
-		(unit 1)
-		(exclude_from_sim no)
-		(in_bom yes)
-		(on_board yes)
-		(dnp no)
-		(fields_autoplaced yes)
-		(property "Reference" "BT1"
-			(at 196.85 41.3384 0)
-			(effects
-				(font
-					(size 1.27 1.27)
-				)
-				(justify left)
-			)
-		)
-		(property "Value" "Battery_Cell"
-			(at 196.85 43.8784 0)
-			(effects
-				(font
-					(size 1.27 1.27)
-				)
-				(justify left)
-			)
-		)
-		(property "Footprint" ""
-			(at 193.04 42.926 90)
-			(effects
-				(font
-					(size 1.27 1.27)
-				)
-				(hide yes)
-			)
-		)
-		(property "Datasheet" "~"
-			(at 193.04 42.926 90)
-			(effects
-				(font
-					(size 1.27 1.27)
-				)
-				(hide yes)
-			)
-		)
-		(property "Description" "Single-cell battery"
-			(at 193.04 44.45 0)
-			(effects
-				(font
-					(size 1.27 1.27)
-				)
-				(hide yes)
-			)
-		)
-		(pin "2"
-		)
-		(pin "1"
-		)
-		(instances
-			(project ""
-				(path "/499b7f21-0212-4c70-b513-805f31ce0850"
-					(reference "BT1")
-					(unit 1)
-				)
-			)
-		)
-	)
-	(symbol
 		(lib_id "Device:LED")
 		(at 186.69 111.76 270)
@@
 	)
 	(symbol
+		(lib_id "easyeda2kicad:XDM254-1-02-W-8.5-G0")
+		(at 198.12 43.18 0)
+		(unit 1)
+		(exclude_from_sim no)
+		(in_bom yes)
+		(on_board yes)
+		(dnp no)
+		(fields_autoplaced yes)
+		(property "Reference" "U6"
+			(at 201.93 41.9099 0)
+			(effects
+				(font
+					(size 1.27 1.27)
+				)
+				(justify left)
+			)
+		)
+		(property "Value" "XDM254-1-02-W-8.5-G0"
+			(at 201.93 44.4499 0)
+			(effects
+				(font
+					(size 1.27 1.27)
+				)
+				(justify left)
+			)
+		)
+		(property "Footprint" "easyeda2kicad:HDR-TH_2P-P2.54-H-F-W10.0-N"
+			(at 198.12 52.07 0)
+			(effects
+				(font
+					(size 1.27 1.27)
+				)
+				(hide yes)
+			)
+		)
+		(property "Datasheet" ""
+			(at 198.12 43.18 0)
+			(effects
+				(font
+					(size 1.27 1.27)
+				)
+				(hide yes)
+			)
+		)
+		(property "Description" ""
+			(at 198.12 43.18 0)
+			(effects
+				(font
+					(size 1.27 1.27)
+				)
+				(hide yes)
+			)
+		)
+		(property "LCSC Part" "C19268733"
+			(at 198.12 54.61 0)
+			(effects
+				(font
+					(size 1.27 1.27)
+				)
+				(hide yes)
+			)
+		)
+		(pin "1"
+		)
+		(pin "2"
+		)
+		(instances
+			(project ""
+				(path "/499b7f21-0212-4c70-b513-805f31ce0850"
+					(reference "U6")
+					(unit 1)
+				)
+			)
+		)
+	)
+	(symbol
 		(lib_id "easyeda2kicad:LGS63042")
 		(at 295.91 114.3 180)
@@
 	(symbol
 		(lib_id "Device:D")
-		(at 124.46 17.78 180)
+		(at 125.73 16.51 180)
 		(unit 1)
 		(exclude_from_sim no)
@@
 		(fields_autoplaced yes)
 		(property "Reference" "D4"
-			(at 124.46 11.43 0)
+			(at 125.73 10.16 0)
 			(effects
 				(font
@@
 		)
 		(property "Value" "D"
-			(at 124.46 13.97 0)
+			(at 125.73 12.7 0)
 			(effects
 				(font
@@
 			)
 		)
-		(property "Footprint" ""
-			(at 124.46 17.78 0)
+		(property "Footprint" "Diode_SMD:D_SMA"
+			(at 125.73 16.51 0)
 			(effects
 				(font
@@
 		)
 		(property "Datasheet" "~"
-			(at 124.46 17.78 0)
+			(at 125.73 16.51 0)
 			(effects
 				(font
@@
 		)
 		(property "Description" "Diode"
-			(at 124.46 17.78 0)
+			(at 125.73 16.51 0)
 			(effects
 				(font
@@
 		)
 		(property "Sim.Device" "D"
-			(at 124.46 17.78 0)
+			(at 125.73 16.51 0)
 			(effects
 				(font
@@
 		)
 		(property "Sim.Pins" "1=K 2=A"
-			(at 124.46 17.78 0)
+			(at 125.73 16.51 0)
+			(effects
+				(font
+					(size 1.27 1.27)
+				)
+				(hide yes)
+			)
+		)
+		(property "LCSC" "C5154212"
+			(at 125.73 16.51 0)
 			(effects
 				(font
