File: led-strip-esphome/led-strip-esphome.kicad_pcb (KiCad board)
At the start: 2 copper layers, 46 parts, among them Q1 FS8205A_C2830320, U1 TP4056_C725790, U2 BL8072COTR33, U3 AI-WB2-12F, U4 LGS63042, U5 DW01A, U6 XDM254-1-02-W-8.5-G0

Commit message: routing
Parts:
- added SW1: TS-1002S-04526C, easyeda2kicad:SW-SMD_4P-L6.0-W6.0-P4.50-LS9.0-2, F.Cu at (233.9, 23.2)
- moved D4 87.1 mm to (52.5, 37.5), turned to 180 degrees
- moved R11 55.9 mm to (182.5, 40.5), turned to 180 degrees
- moved U4 0.98 mm to (150.1, 52.9)
Connections:
- U3 pad 10: unconnected-(U3-IO4-Pad10) -> Net-(U3-IO4)
Routing:
- net /3V~4.2V Out: track 0.00 -> 135.2 mm
- net Net-(D4-A): track 4.71 -> 17.9 mm
- net GND: track 38.6 -> 41.2 mm
- net Net-(U5-CS): vias 0 -> 1

Commit message: finishing
Parts:
- D12, L1, U3: moved to B.Cu
- R11, R4: moved to F.Cu
- moved C5 112.1 mm to (176.1, 53.0)
- moved C6 111.4 mm to (173.0, 55.5)
- moved R8 105.5 mm to (169.0, 43.0), turned to 90 degrees
- moved D13 92.5 mm to (172.0, 47.4), turned to 90 degrees
- moved D16 85.7 mm to (152.0, 47.4), turned to 90 degrees
- moved D14 82.5 mm to (162.0, 47.4), turned to 90 degrees
- moved D6 68.4 mm to (142.0, 47.4), turned to 90 degrees
- moved C3 61.6 mm to (177.5, 41.5), turned to 180 degrees
- moved C4 61.5 mm to (177.5, 39.0), turned to 180 degrees
- moved R4 58.9 mm to (181.0, 41.9), turned to -90 degrees
- moved D7 58.1 mm to (132.0, 47.4), turned to 90 degrees
- moved D18 53.1 mm to (32.0, 47.4), turned to 90 degrees
- moved D8 48.1 mm to (122.0, 47.4), turned to 90 degrees
- moved D1 43.8 mm to (42.0, 47.4), turned to 90 degrees
- moved D10 43.5 mm to (112.0, 47.4), turned to 90 degrees
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Routing:
- net GND: track 41.2 -> 254.5 mm, vias 0 -> 4
- net Net-(D1-A): track 0.00 -> 165.0 mm, vias 0 -> 2
- net Net-(D1-K): track 0.00 -> 148.1 mm, vias 0 -> 1
- net VCC: track 23.6 -> 115.9 mm, vias 0 -> 4
- net TX: track 0.00 -> 51.1 mm
- net RX: track 0.00 -> 46.8 mm
- net /3V~4.2V Out: track 135.2 -> 175.6 mm, vias 0 -> 1
- net Net-(U3-IO14): track 0.00 -> 28.9 mm, vias 0 -> 1
- net Net-(U1-~{STDBY}): track 152.2 -> 173.7 mm
- net Net-(U1-~{CHRG}): track 153.6 -> 175.2 mm
- net Net-(D12-A): track 0.00 -> 18.7 mm, vias 0 -> 1
- net Net-(U3-IO4): track 0.00 -> 11.9 mm, vias 0 -> 1
- net +: track 35.1 -> 41.6 mm
- net Net-(D2-A): track 30.0 -> 36.0 mm, vias 0 -> 1
- net Net-(U5-CS): track 0.00 -> 4.53 mm
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Other:
- board outline added: 219 x 28 mm

Commit message: finished
Routing:
- net Net-(D2-A): track 36.0 -> 196.3 mm, vias 1 -> 3
- net GND: track 254.5 -> 301.7 mm, vias 4 -> 6
- net /3V~4.2V Out: track 175.6 -> 171.4 mm
- net Net-(Q1-G2): track 8.57 -> 10.2 mm
- net +: track 41.6 -> 42.2 mm
Other:
- board size 219 x 28 mm -> 220 x 28 mm

Commit message: update
Routing:
- added copper zone on B.Cu, net GND
- added copper zone on F.Cu, net GND
Changed lines of the file:
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@@
 		(at 218.5 47)
 		(property "Reference" "SW1"
-			(at 0 -6.25 360)
+			(at 0 -6.25 0)
 			(layer "F.SilkS")
 			(effects
@@
 		)
 		(property "Value" "TS-1002S-04526C"
-			(at 0 6.25 360)
+			(at 0 6.25 0)
 			(layer "F.Fab")
 			(effects
@@
 		)
 		(property "Footprint" "easyeda2kicad:SW-SMD_4P-L6.0-W6.0-P4.50-LS9.0-2"
-			(at 0 0 360)
+			(at 0 0 0)
 			(layer "F.Fab")
 			(hide yes)
@@
 		)
 		(property "Datasheet" "https://lcsc.com/product-detail/Tactile-Switches_XUNPU-TS-1002S-04526C_C455109.html"
-			(at 0 0 360)
+			(at 0 0 0)
 			(layer "F.Fab")
 			(hide yes)
@@
 		)
 		(property "Description" ""
-			(at 0 0 360)
+			(at 0 0 0)
 			(layer "F.Fab")
 			(hide yes)
@@
 		)
 		(fp_text user "${REFERENCE}"
-			(at 0 0 360)
+			(at 0 0 0)
 			(layer "F.Fab")
 			(effects
@@
 		(tags "capacitor")
 		(property "Reference" "C5"
-			(at 0 -1.68 360)
+			(at 0 -1.68 0)
 			(layer "F.SilkS")
 			(effects
@@
 		)
 		(property "Value" "4.7uF"
-			(at 0 1.68 360)
+			(at 0 1.68 0)
 			(layer "F.Fab")
 			(effects
@@
 		)
 		(fp_text user "${REFERENCE}"
-			(at 0 0 360)
+			(at 0 0 0)
 			(layer "F.Fab")
 			(effects
@@
 		(tags "capacitor")
 		(property "Reference" "C2"
-			(at 0 1.68 360)
+			(at 0 1.68 0)
 			(layer "B.SilkS")
 			(effects
@@
 		)
 		(property "Value" "10uF"
-			(at 0 -1.68 360)
+			(at 0 -1.68 0)
 			(layer "B.Fab")
 			(effects
@@
 		)
 		(fp_text user "${REFERENCE}"
-			(at 0 0 360)
+			(at 0 0 0)
 			(layer "B.Fab")
 			(effects
@@
 		(tags "LED")
 		(property "Reference" "R7"
-			(at 2.52869 0 360)
+			(at 2.52869 0 0)
 			(layer "B.SilkS")
 			(effects
@@
 		)
 		(property "Value" "5.11k"
-			(at 0 -1.65 360)
+			(at 0 -1.65 0)
 			(layer "B.Fab")
 			(effects
@@
 		)
 		(fp_text user "${REFERENCE}"
-			(at 0 0 360)
+			(at 0 0 0)
 			(layer "B.Fab")
 			(effects
@@
 		(tags "capacitor")
 		(property "Reference" "C3"
-			(at 3 0 360)
+			(at 3 0 0)
 			(layer "B.SilkS")
 			(effects
@@
 		)
 		(property "Value" "1uF"
-			(at 0 -1.68 360)
+			(at 0 -1.68 0)
 			(layer "B.Fab")
 			(effects
@@
 		)
 		(fp_text user "${REFERENCE}"
-			(at 0 0 360)
+			(at 0 0 0)
 			(layer "B.Fab")
 			(effects
@@
 		(tags "LED")
 		(property "Reference" "R2"
-			(at -0.03381 -2 360)
+			(at -0.03381 -2 0)
 			(layer "B.SilkS")
 			(effects
@@
 		)
 		(property "Value" "210"
-			(at 0 -1.65 360)
+			(at 0 -1.65 0)
 			(layer "B.Fab")
 			(effects
@@
 		)
 		(fp_text user "${REFERENCE}"
-			(at 0 0 360)
+			(at 0 0 0)
 			(layer "B.Fab")
 			(effects
@@
 		(tags "LED")
 		(property "Reference" "R5"
-			(at 2.59119 0 360)
+			(at 2.59119 0 0)
 			(layer "B.SilkS")
 			(effects
@@
 		)
 		(property "Value" "1M"
-			(at 0 -1.65 360)
+			(at 0 -1.65 0)
 			(layer "B.Fab")
 			(effects
@@
 		)
 		(fp_text user "${REFERENCE}"
-			(at 0 0 360)
+			(at 0 0 0)
 			(layer "B.Fab")
 			(effects
@@
 		(tags "capacitor")
 		(property "Reference" "C1"
-			(at 4.05 0 360)
+			(at 4.05 0 0)
 			(layer "B.SilkS")
 			(effects
@@
 		)
 		(property "Value" "10uF"
-			(at 0 -1.68 360)
+			(at 0 -1.68 0)
 			(layer "B.Fab")
 			(effects
@@
 		)
 		(fp_text user "${REFERENCE}"
-			(at 0 0 360)
+			(at 0 0 0)
 			(layer "B.Fab")
 			(effects
@@
 		(tags "smd inductor dlg-0403")
 		(property "Reference" "L1"
-			(at 0 3.2 360)
+			(at 0 3.2 0)
 			(layer "B.SilkS")
 			(effects
@@
 		)
 		(property "Value" "10uH"
-			(at 0 -3.2 360)
+			(at 0 -3.2 0)
 			(layer "B.Fab")
 			(effects
@@
 		)
 		(fp_text user "${REFERENCE}"
-			(at 0 0 360)
+			(at 0 0 0)
 			(layer "B.Fab")
 			(effects
@@
 		(tags "LED")
 		(property "Reference" "D3"
-			(at 0 1.43 360)
+			(at 0 1.43 0)
 			(layer "B.SilkS")
 			(effects
@@
 		)
 		(property "Value" "LED"
-			(at 0 -1.43 360)
+			(at 0 -1.43 0)
 			(layer "B.Fab")
 			(effects
@@
 		)
 		(fp_text user "${REFERENCE}"
-			(at 0 0 360)
+			(at 0 0 0)
 			(layer "B.Fab")
 			(effects
@@
 		(tags "LED")
 		(property "Reference" "R3"
-			(at 0 1.65 360)
+			(at 0 1.65 0)
 			(layer "B.SilkS")
 			(effects
@@
 		)
 		(property "Value" "210"
-			(at 0 -1.65 360)
+			(at 0 -1.65 0)
 			(layer "B.Fab")
 			(effects
@@
 		)
 		(fp_text user "${REFERENCE}"
-			(at 0 0 360)
+			(at 0 0 0)
 			(layer "B.Fab")
 			(effects
@@
 		(tags "LED")
 		(property "Reference" "D2"
-			(at 0 -1.5 360)
+			(at 0 -1.5 0)
 			(layer "B.SilkS")
 			(effects
@@
 		)
 		(property "Value" "LED"
-			(at 0 -1.43 360)
+			(at 0 -1.43 0)
 			(layer "B.Fab")
 			(effects
@@
 		)
 		(fp_text user "${REFERENCE}"
-			(at 0 0 360)
+			(at 0 0 0)
 			(layer "B.Fab")
 			(effects
@@
 		(tags "LED")
 		(property "Reference" "R6"
-			(at 2.52869 0 360)
+			(at 2.52869 0 0)
 			(layer "B.SilkS")
 			(effects
@@
 		)
 		(property "Value" "5.11k"
-			(at 0 -1.65 360)
+			(at 0 -1.65 0)
 			(layer "B.Fab")
 			(effects
@@
 		)
 		(fp_text user "${REFERENCE}"
-			(at 0 0 360)
+			(at 0 0 0)
 			(layer "B.Fab")
 			(effects
@@
 		(tags "capacitor")
 		(property "Reference" "C4"
-			(at -3 0 360)
+			(at -3 0 0)
 			(layer "B.SilkS")
 			(effects
@@
 		)
 		(property "Value" "1uF"
-			(at 0 -1.68 360)
+			(at 0 -1.68 0)
 			(layer "B.Fab")
 			(effects
@@
 		)
 		(fp_text user "${REFERENCE}"
-			(at 0 0 360)
+			(at 0 0 0)
 			(layer "B.Fab")
 			(effects
@@
 		(tags "Diode SMA (DO-214AC)")
 		(property "Reference" "D4"
-			(at 0 2.5 360)
+			(at 0 2.5 0)
 			(layer "B.SilkS")
 			(effects
@@
 		)
 		(property "Value" "D"
-			(at 0 -2.6 360)
+			(at 0 -2.6 0)
 			(layer "B.Fab")
 			(effects
@@
 		)
 		(fp_text user "${REFERENCE}"
-			(at 0 2.5 360)
+			(at 0 2.5 0)
 			(layer "B.Fab")
 			(effects
@@
 		(net 49)
 	)
+	(zone
+		(net 5)
+		(net_name "GND")
+		(layers "F&B.Cu")
+		(hatch edge 0.5)
+		(connect_pads
+			(clearance 0.5)
+		)
+		(min_thickness 0.25)
+		(filled_areas_thickness no)
+		(fill yes
+			(thermal_gap 0.5)
+			(thermal_bridge_width 0.5)
+		)
+		(polygon
+			(pts
+				(xy 14.5 33) (xy 14.5 61) (xy 234.5 61) (xy 234.5 33)
+			)
+		)
+	)
 )
